Commit message: Add dummy link to agv_base.urdf.xacro root

File: agv_description/urdf/agv_base.urdf.xacro (robot description, xacro)
@@ -2,4 +2,10 @@
 <robot xmlns:xacro="http://ros.org/wiki/xacro">
   <xacro:macro name="agv_base" >
+    <link name="base_footprint"/>
+    <joint name="base_joint" type="fixed">
+      <parent link="base_footprint"/>
+      <child link="base_link"/>
+      <origin xyz="0.0 0.0 0.010" rpy="0 0 0"/>
+    </joint>
     <link name='base_link'>
       <origin xyz="0 0 0" rpy=" 0 0 0"/>
