Commit message: Resize agv to 4000mm x 1200mm

File: agv_description/urdf/agv.urdf.xacro (robot description, xacro)
@@ -8,18 +8,6 @@
 	<xacro:include filename="$(find agv_description)/urdf/agv_ir.urdf.xacro"/>
 	<xacro:agv_base />
-	<xacro:agv_ir base_link="base_link" link_name="ir1" xyz_ir="0.505 0.215 -0.03" rpy_ir="0 0 0" />
-	<xacro:agv_ir base_link="base_link" link_name="ir2" xyz_ir="0.20 0.355 -0.068" rpy_ir="0 0 1.570796" />
-	<xacro:agv_ir base_link="base_link" link_name="ir3" xyz_ir="-0.20 0.355 -0.068" rpy_ir="0 0 1.570796" />
-	<xacro:agv_ir base_link="base_link" link_name="ir4" xyz_ir="-0.505 0.215 -0.005" rpy_ir="0 0 3.14159" />
-	<xacro:agv_ir base_link="base_link" link_name="ir5" xyz_ir="-0.505 -0.215 -0.005" rpy_ir="0 0 3.14159" />
-	<xacro:agv_ir base_link="base_link" link_name="ir6" xyz_ir="-0.20 -0.355 -0.068" rpy_ir="0 0 -1.570796" />
-	<xacro:agv_ir base_link="base_link" link_name="ir7" xyz_ir="0.20 -0.355 -0.068" rpy_ir="0 0 -1.570796" />
-	<xacro:agv_ir base_link="base_link" link_name="ir8" xyz_ir="0.503 -0.215 -0.03" rpy_ir="0 0 0" />
-	<xacro:agv_wheel xyz_hub="0 -0.30 -0.06" rpy_hub="0 0 0" side="left"/>
-	<xacro:agv_wheel xyz_hub="0 0.30 -0.06" rpy_hub="0 0 0" side="right"/>
-	<xacro:agv_swivel xyz_caster="0.37 -0.22 -0.048" rpy_caster="0 0 0" side="front_right"/>
-	<xacro:agv_swivel xyz_caster="0.37 0.22 -0.048" rpy_caster="0 0 0" side="front_left"/>
-	<xacro:agv_swivel xyz_caster="-0.37 -0.22 -0.048" rpy_caster="0 0 0" side="back_right"/>
-	<xacro:agv_swivel xyz_caster="-0.37 0.22 -0.048" rpy_caster="0 0 0" side="back_left"/>
+	<xacro:agv_ir base_link="base_link" link_name="ir1" xyz_ir="2.02 0.3655 -0.03" rpy_ir="0 0 0" />
+	<xacro:a표로 잡고 설정v_swivel xyz_caster="-1.48 0.374 -0.048" rpy_caster="0 0 0" side="back_left"/>
 	<!-- Motor plugin -->
 	<xacro:agv_diff_drive />

File: agv_description/urdf/agv_base.urdf.xacro (robot description, xacro)
@@ -13,5 +13,5 @@
         <origin xyz="0 0 -0.1625" rpy=" 0 0 0"/>
         <geometry>
-          <mesh filename="package://agv_description/meshes/OTAv07_meshes/OTA-v0.7.stl" scale="0.001 0.001 0.001"/>
+          <mesh filename="package://agv_description/meshes/OTAv07_meshes/OTA-v0.7.stl" scale="0.004 0.0017 0.001"/>
         </geometry>
       </visual>
@@ -19,6 +19,6 @@
         <origin xyz="0 0 -0.075" rpy=" 0 0 0"/>
         <geometry>
-          <!--<mesh filename="package://agv_description/meshes/OTAv07_meshes/OTA-v0.7.stl" scale="0.001 0.001 0.001"/> -->
-          <box size="1.02 0.72 0.14"/>
+          <mesh filename="package://agv_description/meshes/OTAv07_meshes/OTA-v0.7.stl" scale="0.004 0.0017 0.001"/>
+          <!-- <box size="1.02 0.72 0.14"/> -->
         </geometry>
       </collision>
@@ -107,5 +107,5 @@
       <parent link="base_link"/>
       <child link="zed_camera"/>
-      <origin xyz="0.49 0 0.175" rpy="0 0 0" />
+      <origin xyz="2.03 0 0.175" rpy="0 0 0" />
     </joint>
     <gazebo reference="zed_camera">

File: agv_description/urdf/agv_plugin.urdf.xacro (robot description, xacro)
@@ -22,5 +22,5 @@
         <leftJoint>wheel_right_base</leftJoint>
         <rightJoint>wheel_left_base</rightJoint>
-        <wheelSeparation>0.60</wheelSeparation>
+        <wheelSeparation>1.02</wheelSeparation>
         <wheelDiameter>0.20</wheelDiameter>
         <wheelTorque>20</wheelTorque>
